Commit message: adding gps plugin

File: src/description/robot_description.urdf (robot description, URDF)
Before this commit: robot sam_bot, 7 links, 6 joints
Links:
- added link gps_link, mass 0.035; collision box size=0.015 -0.4 0.044; visual box size=0.0 -0.4 0.044
Joints:
- added joint gps_joint: type fixed, parent base_link, child gps_link, origin xyz=0.0 0 0.0 rpy=0 0 0

Commit message: removing pyc and adding ekf to the launch file

File: src/description/robot_description.urdf (robot description, URDF)
Before this commit: robot sam_bot, 8 links, 7 joints
Links:
- removed link lidar_link
- link gps_link: mass 0.035 -> 0.125; geometry collision cylinder length=0.055 radius=0.0508; visual cylinder length=0.055 radius=0.0508
Joints:
- removed joint lidar_joint
- joint gps_joint: origin xyz=0.0 0 0.0 rpy=0 0 0 -> xyz=0 0 0.12 rpy=0 0 0
